Commit message: calibration script update

File: nico_alljoints.urdf (robot description, URDF)
Before this commit: robot nico_upper_rh6d, 23 links, 22 joints
Links:
- added link endeffector; visual sphere radius=0.005s
Joints:
- added joint endeffector_joint: type fixed, parent right_palm, child endeffector, origin xyz=0.00 -0.02 -0.11 rpy=0 0 0

Commit message: calibration procedure for left and right hand with results

File: nico_alljoints.urdf (robot description, URDF)
Before this commit: robot nico_upper_rh6d, 24 links, 23 joints
Links:
- added link endeffectol; visual sphere radius=0.007
- link endeffector: geometry visual sphere radius=0.007
Joints:
- added joint endeffectol_joint: type fixed, parent left_palm, child endeffectol, origin xyz=0.00 -0.02 -0.11 rpy=0 0 0

Commit message: nico alljoints urdf updated according nohands urdf - URDF finetuned

File: nico_alljoints.urdf (robot description, URDF)
Before this commit: robot nico_upper_rh6d, 25 links, 24 joints
Joints:
- joint head_z: origin xyz=-0.025 0.005 0.23 rpy=0 0 0 -> xyz=-0.025 0.000 0.23 rpy=0 0 0
- joint l_shoulder_y: limit lower=-0.5236 upper=3.1416 effort=30 velocity=1 -> lower=-1.5707 upper=3.1416 effort=30 velocity=1
- joint l_shoulder_z: origin xyz=0.005 0.05 0.23 rpy=0 0 0 -> xyz=0.000 0.040 0.23 rpy=0 0 0
- joint r_shoulder_y: limit lower=0 upper=3.1416 effort=30 velocity=1 -> lower=-1.5707 upper=3.1416 effort=30 velocity=1
- joint r_shoulder_z: origin xyz=0.005 -0.045 0.23 rpy=0 0 0 -> xyz=0.000 -0.040 0.23 rpy=0 0 0
