Commit message: manual calibrtion - WORKING

File: calibration.urdf (robot description, URDF)
Before this commit: robot nico_upper_rh6d, 20 links, 17 joints
Links:
- removed link endeffectol
- removed link endeffector
Joints:
- removed joint head_y_rjoint
- removed joint head_z_rjoint
- removed joint l_shoulder_y_rjoint
- removed joint l_upperarm_x
- added joint head_y: type revolute, parent neck, child head, origin xyz=0 0.0 0.105 rpy=0 0 0, axis 0 -1 0, limit lower=-0.8726 upper=0.4363 effort=30 velocity=1
- added joint head_z: type revolute, parent torso, child neck, origin xyz=-0.025 0.005 0.23 rpy=0 0 0, axis 0 0 1, limit lower=-1.5708 upper=1.5708 effort=30 velocity=1
- added joint l_arm_x: type revolute, parent left_collarbone, child left_upper_arm, origin xyz=0.00 0.073 -0.023 rpy=0 0 0, axis 1 0 0, limit lower=0 upper=1.2217 effort=30 velocity=1
- added joint l_shoulder_y: type revolute, parent left_shoulder, child left_collarbone, origin xyz=-0.021 0.023 0.033 rpy=0 0 0, axis 0 -1 0, limit lower=-0.5236 upper=3.1416 effort=30 velocity=1
- joint grippel_: type revolute -> fixed
- joint r_indexfinger_x: limit (none) -> lower=-2.57 upper=0 effort=30 velocity=1

Commit message: urdf calibration update

File: calibration.urdf (robot description, URDF)
Before this commit: robot nico_upper_rh6d, 18 links, 17 joints
Links:
- removed link grippel
- removed link gripper
- added link l_indexfinger, mass 0.000009; collision mesh filename=mesh/finger.stl; visual mesh filename=mesh/finger.stl
- added link l_littlefinger, mass 0.000009; collision mesh filename=mesh/finger.stl; visual mesh filename=mesh/finger.stl
- added link l_middlefinger, mass 0.000009; collision mesh filename=mesh/finger.stl; visual mesh filename=mesh/finger.stl
- added link r_indexfinger, mass 0.000009; collision mesh filename=mesh/finger.stl; visual mesh filename=mesh/finger.stl
- added link r_littlefinger, mass 0.000009; collision mesh filename=mesh/finger.stl; visual mesh filename=mesh/finger.stl
- added link r_middlefinger, mass 0.000009; collision mesh filename=mesh/finger.stl; visual mesh filename=mesh/finger.stl
- added link sight, mass 0.000009; visual cylinder length=0.6 radius=0.001
Joints:
- removed joint grippel_
- added joint eyesight: type fixed, parent head, child sight, origin xyz=0 0.0 0.0 rpy=0 0 0, axis 0 0 0, limit lower=-0.8726 upper=0.4363 effort=30 velocity=1
- added joint l_indexfiner_x: type fixed, parent left_palm, child l_indexfinger, origin xyz=0.00 -0.02 -0.06 rpy=0 0 0, axis 0 1 0, limit lower=0 upper=2.57 effort=30 velocity=1
- added joint l_litlefinger_x: type fixed, parent left_palm, child l_littlefinger, origin xyz=0.00 0.02 -0.06 rpy=0 0 0, axis 0 1 0, limit lower=-2.57 upper=0 effort=30 velocity=1
- added joint l_middlefinger_x: type fixed, parent left_palm, child l_middlefinger, origin xyz=0 0 -0.06 rpy=0 0 0, axis 0 1 0, limit lower=-2.57 upper=0 effort=30 velocity=1
- added joint r_litlefinger_x: type fixed, parent right_palm, child r_littlefinger, origin xyz=0.00 0.02 -0.06 rpy=0 0 0, axis 0 1 0, limit lower=-2.57 upper=0 effort=30 velocity=1
- added joint r_middlefinger_x: type fixed, parent right_palm, child r_middlefinger, origin xyz=0 0 -0.06 rpy=0 0 0, axis 0 1 0, limit lower=-2.57 upper=0 effort=30 velocity=1
- joint l_shoulder_z: axis 0 0 1 -> 0 0 -1
- joint l_wrist_z: axis 0 0 1 -> 0 0 -1
- joint r_indexfinger_x: child gripper -> r_indexfinger; origin xyz=0.00 -0.02 -0.06 rpy=0 -1 0 -> xyz=0.00 -0.02 -0.06 rpy=0 0 0; type revolute -> fixed

Commit message: urdf elbow position update for callibration

File: calibration.urdf (robot description, URDF)
Before this commit: robot nico_upper_rh6d, 23 links, 22 joints
Joints:
- joint l_elbow_y: origin xyz=0.0 0 -0.17 rpy=0 3.14 0 -> xyz=0.0 0 -0.17 rpy=0 -1.57 0
- joint r_elbow_y: origin xyz=0.0 0 -0.17 rpy=0 3.14 0 -> xyz=0.0 0 -0.17 rpy=0 -1.57 0

Commit message: all urdf UPDATED - will be merged in next commit

File: calibration.urdf (robot description, URDF)
Before this commit: robot nico_upper_rh6d, 23 links, 22 joints
Joints:
- joint head_z: limit lower=-1.5708 upper=1.5708 effort=30 velocity=1 -> lower=-1.5707 upper=1.5707 effort=30 velocity=1; origin xyz=-0.025 0.005 0.23 rpy=0 0 0 -> xyz=-0.025 0.000 0.23 rpy=0 0 0
- joint l_elbow_y: limit lower=0.8726 upper=3.1416 effort=30 velocity=1 -> lower=-0.6981 upper=1.5707 effort=30 velocity=1; origin xyz=0.0 0 -0.17 rpy=0 -1.57 0 -> xyz=0.0 0 -0.17 rpy=0 -1.5707 0
- joint l_shoulder_y: limit lower=-0.5236 upper=3.1416 effort=30 velocity=1 -> lower=-1.5707 upper=3.1416 effort=30 velocity=1
- joint l_shoulder_z: origin xyz=0.005 0.05 0.23 rpy=0 0 0 -> xyz=0.000 0.040 0.23 rpy=0 0 0
- joint l_wrist_z: limit lower=-1.571 upper=1.571 effort=30 velocity=1 -> lower=-1.5707 upper=1.5707 effort=30 velocity=1; origin xyz=0 0 -0.105 rpy=0 0 1.57 -> xyz=0 0 -0.105 rpy=0 0 1.5707
- joint r_elbow_y: limit lower=0.8726 upper=3.1416 effort=30 velocity=1 -> lower=-0.6981 upper=1.5707 effort=30 velocity=1; origin xyz=0.0 0 -0.17 rpy=0 -1.57 0 -> xyz=0.0 0 -0.17 rpy=0 -1.5707 0
- joint r_shoulder_y: limit lower=0 upper=3.1416 effort=30 velocity=1 -> lower=-1.5707 upper=3.1416 effort=30 velocity=1
- joint r_shoulder_z: origin xyz=0.005 -0.045 0.23 rpy=0 0 0 -> xyz=0.000 -0.040 0.23 rpy=0 0 0
- joint r_wrist_z: limit lower=-1.57079633 upper=1.57079633 effort=30 velocity=1 -> lower=-1.5707 upper=1.5707 effort=30 velocity=1; origin xyz=0 0 -0.105 rpy=0 0 1.57 -> xyz=0 0 -0.105 rpy=0 0 1.5707

File: nico_alljoints.urdf (robot description, URDF)
Before this commit: robot nico_upper_rh6d, 25 links, 24 joints
Joints:
- joint head_z: limit lower=-1.5708 upper=1.5708 effort=30 velocity=1 -> lower=-1.5707 upper=1.5707 effort=30 velocity=1
- joint l_elbow_y: limit lower=0.8726 upper=3.1416 effort=30 velocity=1 -> lower=-0.6981 upper=1.5707 effort=30 velocity=1; origin xyz=0.0 0 -0.17 rpy=0 3.14 0 -> xyz=0.0 0 -0.17 rpy=0 -1.5707 0
- joint l_wrist_z: limit lower=-1.571 upper=1.571 effort=30 velocity=1 -> lower=-1.5707 upper=1.5707 effort=30 velocity=1; origin xyz=0 0 -0.105 rpy=0 0 1.57 -> xyz=0 0 -0.105 rpy=0 0 1.5707
- joint r_elbow_y: limit lower=0.8726 upper=3.1416 effort=30 velocity=1 -> lower=-0.6981 upper=1.5707 effort=30 velocity=1; origin xyz=0.0 0 -0.17 rpy=0 3.14 0 -> xyz=0.0 0 -0.17 rpy=0 -1.5707 0
- joint r_wrist_z: limit lower=-1.57079633 upper=1.57079633 effort=30 velocity=1 -> lower=-1.5707 upper=1.5707 effort=30 velocity=1; origin xyz=0 0 -0.105 rpy=0 0 1.57 -> xyz=0 0 -0.105 rpy=0 0 1.5707

File: nico_upper_rh6d_l.urdf (robot description, URDF)
Before this commit: robot nico_upper_rh6d, 20 links, 19 joints
Links:
- added link sight, mass 0.000009; visual cylinder length=0.6 radius=0.001
- link endeffectol: mass None -> 0.000009
- link endeffector: mass None -> 0.000009
- link torso: mass None -> 0.090439
Joints:
- removed joint gripper_rjoint
- added joint eyesight: type fixed, parent head, child sight, origin xyz=0 0.0 0.0 rpy=0 0 0, axis 0 0 0, limit lower=-0.8726 upper=0.4363 effort=30 velocity=1
- added joint r_indexfinger_x: type fixed, parent right_palm, child gripper, origin xyz=0.00 -0.02 -0.06 rpy=0 -1 0, axis 0 1 0
- joint head_y_rjoint: axis 0 1 0 -> 0 -1 0
- joint head_z_rjoint: limit lower=-1.5708 upper=1.5708 effort=30 velocity=1 -> lower=-1.5707 upper=1.5707 effort=30 velocity=1; origin xyz=-0.025 0.005 0.23 rpy=0 0 0 -> xyz=-0.025 0.000 0.23 rpy=0 0 0
- joint l_elbow_y_rjoint: limit lower=0.8726 upper=3.1416 effort=30 velocity=1 -> lower=-0.6981 upper=1.5707 effort=30 velocity=1; origin xyz=0.0 0 -0.17 rpy=0 3.14 0 -> xyz=0.0 0 -0.17 rpy=0 -1.5707 0
- joint l_shoulder_y_rjoint: limit lower=-0.5236 upper=3.1416 effort=30 velocity=1 -> lower=-1.5707 upper=3.1416 effort=30 velocity=1
- joint l_shoulder_z_rjoint: axis 0 0 1 -> 0 0 -1; origin xyz=0.005 0.05 0.23 rpy=0 0 0 -> xyz=0.000 0.040 0.23 rpy=0 0 0
- joint l_wrist_z_rjoint: axis 0 0 1 -> 0 0 -1; limit lower=-1.571 upper=1.571 effort=30 velocity=1 -> lower=-1.5707 upper=1.5707 effort=30 velocity=1; origin xyz=0 0 -0.105 rpy=0 0 1.57 -> xyz=0 0 -0.105 rpy=0 0 1.5707
- joint r_elbow_y_rjoint: limit lower=0.8726 upper=3.1416 effort=30 velocity=1 -> lower=-0.6981 upper=1.5707 effort=30 velocity=1; origin xyz=0.0 0 -0.17 rpy=0 3.14 0 -> xyz=0.0 0 -0.17 rpy=0 -1.5707 0
- joint r_shoulder_y_rjoint: limit lower=-0.5236 upper=3.1416 effort=30 velocity=1 -> lower=-1.5707 upper=3.1416 effort=30 velocity=1
- joint r_shoulder_z_rjoint: origin xyz=0.005 -0.045 0.23 rpy=0 0 0 -> xyz=0.000 -0.040 0.23 rpy=0 0 0
- joint r_wrist_x_rjoint: axis 0 1 0 -> 0 -1 0; limit lower=-.78 upper=0.78 effort=30 velocity=1 -> lower=-0.785398163 upper=0.785398163 effort=30 velocity=1
- joint r_wrist_z_rjoint: limit lower=-1.571 upper=1.571 effort=30 velocity=1 -> lower=-1.5707 upper=1.5707 effort=30 velocity=1; origin xyz=0 0 -0.105 rpy=0 0 1.57 -> xyz=0 0 -0.105 rpy=0 0 1.5707

File: nico_upper_rh6d_r.urdf (robot description, URDF)
Before this commit: robot nico_upper_rh6d, 20 links, 19 joints
Links:
- added link sight, mass 0.000009; visual cylinder length=0.6 radius=0.001
Joints:
- added joint eyesight: type fixed, parent head, child sight, origin xyz=0 0.0 0.0 rpy=0 0 0, axis 0 0 0, limit lower=-0.8726 upper=0.4363 effort=30 velocity=1
- joint head_y_rjoint: axis 0 1 0 -> 0 -1 0
- joint head_z_rjoint: limit lower=-1.5708 upper=1.5708 effort=30 velocity=1 -> lower=-1.5707 upper=1.5707 effort=30 velocity=1; origin xyz=-0.025 0.005 0.23 rpy=0 0 0 -> xyz=-0.025 0.000 0.23 rpy=0 0 0
- joint l_elbow_y_rjoint: limit lower=0.8726 upper=3.1416 effort=30 velocity=1 -> lower=-0.6981 upper=1.5707 effort=30 velocity=1; origin xyz=0.0 0 -0.17 rpy=0 3.14 0 -> xyz=0.0 0 -0.17 rpy=0 -1.5707 0
- joint l_shoulder_y_rjoint: limit lower=-0.5236 upper=3.1416 effort=30 velocity=1 -> lower=-1.5707 upper=3.1416 effort=30 velocity=1
- joint l_shoulder_z_rjoint: axis 0 0 1 -> 0 0 -1; origin xyz=0.005 0.05 0.23 rpy=0 0 0 -> xyz=0.000 0.040 0.23 rpy=0 0 0
- joint l_wrist_z_rjoint: axis 0 0 1 -> 0 0 -1; limit lower=-1.571 upper=1.571 effort=30 velocity=1 -> lower=-1.5707 upper=1.5707 effort=30 velocity=1; origin xyz=0 0 -0.105 rpy=0 0 1.57 -> xyz=0 0 -0.105 rpy=0 0 1.5707
- joint r_elbow_y: limit lower=0.8726 upper=3.1416 effort=30 velocity=1 -> lower=-0.6981 upper=1.5707 effort=30 velocity=1; origin xyz=0.0 0 -0.17 rpy=0 3.14 0 -> xyz=0.0 0 -0.17 rpy=0 -1.5707 0
- joint r_shoulder_y: limit lower=0 upper=3.1416 effort=30 velocity=1 -> lower=-1.5707 upper=3.1416 effort=30 velocity=1
- joint r_shoulder_z: origin xyz=0.005 -0.045 0.23 rpy=0 0 0 -> xyz=0.000 -0.040 0.23 rpy=0 0 0
- joint r_wrist_z: limit lower=-1.57079633 upper=1.57079633 effort=30 velocity=1 -> lower=-1.5707 upper=1.5707 effort=30 velocity=1; origin xyz=0 0 -0.105 rpy=0 0 1.57 -> xyz=0 0 -0.105 rpy=0 0 1.5707
