Commit message: URDF cleaned and merged - nico-unity.urdf , nico.urdf with fingers, nico...r and l without fingers

File: nico.urdf (robot description, URDF)
Before this commit: robot nico_upper_rh6d, 23 links, 22 joints
Links:
- added link endeffectol; visual sphere radius=0.007
- added link endeffector; visual sphere radius=0.007
Joints:
- added joint endeffectol_joint: type fixed, parent left_palm, child endeffectol, origin xyz=0.00 -0.02 -0.11 rpy=0 0 0
- added joint endeffector_joint: type fixed, parent right_palm, child endeffector, origin xyz=0.00 -0.02 -0.11 rpy=0 0 0
- joint l_elbow_y: limit lower=-0.6981 upper=1.5707 effort=30 velocity=1 -> lower=0.8726 upper=3.1416 effort=30 velocity=1; origin xyz=0.0 0 -0.17 rpy=0 -1.5707 0 -> xyz=0.0 0 -0.17 rpy=0 3.14 0
- joint r_elbow_y: limit lower=-0.6981 upper=1.5707 effort=30 velocity=1 -> lower=0.8726 upper=3.1416 effort=30 velocity=1; origin xyz=0.0 0 -0.17 rpy=0 -1.5707 0 -> xyz=0.0 0 -0.17 rpy=0 3.14 0

File: nico_upper_rh6d_l.urdf (robot description, URDF)
Before this commit: robot nico_upper_rh6d, 21 links, 20 joints
Joints:
- joint l_elbow_y_rjoint: limit lower=-0.6981 upper=1.5707 effort=30 velocity=1 -> lower=0.8726 upper=3.1416 effort=30 velocity=1; origin xyz=0.0 0 -0.17 rpy=0 -1.5707 0 -> xyz=0.0 0 -0.17 rpy=0 3.14 0
- joint r_elbow_y_rjoint: limit lower=-0.6981 upper=1.5707 effort=30 velocity=1 -> lower=0.8726 upper=3.1416 effort=30 velocity=1; origin xyz=0.0 0 -0.17 rpy=0 -1.5707 0 -> xyz=0.0 0 -0.17 rpy=0 3.14 0
- joint r_indexfinger_x: limit (none) -> lower=-2.57 upper=0 effort=30 velocity=1

File: nico_upper_rh6d_r.urdf (robot description, URDF)
Before this commit: robot nico_upper_rh6d, 21 links, 20 joints
Joints:
- joint l_elbow_y_rjoint: limit lower=-0.6981 upper=1.5707 effort=30 velocity=1 -> lower=0.8726 upper=3.1416 effort=30 velocity=1; origin xyz=0.0 0 -0.17 rpy=0 -1.5707 0 -> xyz=0.0 0 -0.17 rpy=0 3.14 0
- joint r_elbow_y: limit lower=-0.6981 upper=1.5707 effort=30 velocity=1 -> lower=0.8726 upper=3.1416 effort=30 velocity=1; origin xyz=0.0 0 -0.17 rpy=0 -1.5707 0 -> xyz=0.0 0 -0.17 rpy=0 3.14 0
- joint r_indexfinger_x: limit (none) -> lower=-2.57 upper=0 effort=30 velocity=1
