Commit message: grasp checking procedure updated - WORKING

File: tiago_dual_mygym.urdf (robot description, URDF)
Before this commit: robot tiago_dual_mygym, 37 links, 36 joints
Links:
- link gripper_right_left_finger_link: geometry collision mesh filename=tiago/gripper_finger_link.stl; visual mesh filename=tiago/gripper_finger_link.stl
- link gripper_right_right_finger_link: geometry collision mesh filename=tiago/gripper_finger_link.stl scale=-1 -1 1; visual mesh filename=tiago/gripper_finger_link.stl scale=-1 -1 1

Commit message: tiago grasp_checker - WORKING

File: tiago_dual_mygym.urdf (robot description, URDF)
Before this commit: robot tiago_dual_mygym, 37 links, 36 joints
Links:
- added link base_footprint2
- link arm_left_1_link: geometry visual mesh filename=tiago/arm_1.stl scale=1 -1 -1
- link arm_right_2_link: geometry visual mesh filename=tiago/arm_2.stl scale=1 1 1
- link arm_right_3_link: geometry visual mesh filename=tiago/arm_3.stl scale=1 1 1
- link arm_right_4_link: geometry visual mesh filename=tiago/arm_4.stl scale=1 1 1
- link arm_right_5_link: geometry visual mesh filename=tiago/arm_5-wrist-2017.stl scale=1 1 1
- link arm_right_6_link: geometry visual mesh filename=tiago//arm_6-wrist-2017.stl scale=1 1 1
- link arm_right_tool_link: geometry visual cylinder length=0.005 radius=0.005
- link base_footprint: mass 1 -> None
- link base_link: mass 28.26649 -> 20.26649
- link gripper_right_link: geometry visual mesh filename=tiago/gripper_link.stl
- link head_1_link: geometry visual mesh filename=tiago/head_1.stl scale=1 1 1
- link head_2_link: geometry visual mesh filename=tiago/head_2.stl scale=1 1 1
- link torso_lift_link: geometry collision mesh filename=tiago/torso_lift_dual_arm.stl scale=1 1 1; visual mesh filename=tiago/torso_lift_dual_arm.stl scale=1 1 1
- link wrist_right_ft_link: geometry visual cylinder length=0.0157 radius=0.0225
- link wrist_right_ft_tool_link: geometry visual cylinder length=0.00975 radius=0.025
Joints:
- added joint baseslide2_rjoint: type prismatic, parent base_footprint, child base_footprint2, origin xyz=0. 0 0 rpy=0 0 0, axis 1 0 0, limit lower=-0.5 upper=0.4 effort=500 velocity=1
- joint arm_left_1_joint: limit lower=-1.1780972451 upper=1.57079632679 effort=43.0 velocity=1.95 -> lower=-1.1780972451 upper=1.57079632679 effort=43.0 velocity=10
- joint baserot_rjoint: limit lower=-1.1780972451 upper=1.57079632679 effort=16 velocity=1.95 -> lower=-1.1780972451 upper=1.57079632679 effort=200 velocity=20; type fixed -> revolute
- joint baseslide_rjoint: limit lower=-0.5 upper=0.5 effort=16 velocity=0.05 -> lower=-0.7 upper=0.35 effort=500 velocity=1; type fixed -> prismatic
