Commit message: error calculation added - distance and quatdiff

File: nico_grasp.urdf (robot description, URDF)
Before this commit: robot nico_upper_rh6d, 27 links, 26 joints
Links:
- link endeffector: geometry visual cylinder length=0.05 radius=0.002
Joints:
- joint endeffector_joint: origin xyz=0.03 0.0 -0.05 rpy=0 0 0 -> xyz=0.03 0.0 -0.05 rpy=3.14 1.57 0
