Commit message: open and close keypress implemented - left hand small bug

File: nico_grasp_right.urdf (robot description, URDF)
Before this commit: robot nico_upper_rh6d, 27 links, 26 joints
Joints:
- joint l_arm_x: type revolute -> fixed
- joint l_elbow_y: type revolute -> fixed
- joint l_shoulder_y: type revolute -> fixed
- joint l_shoulder_z: type revolute -> fixed
- joint l_wrist_z: type revolute -> fixed
