Commit message: grasper updates - left nd right hand switch - left is WIP

File: nico_grasper.urdf (robot description, URDF)
Before this commit: robot nico_upper_rh6d, 27 links, 26 joints
Links:
- added link l_thumb_intermediate_link, mass 0.0000332
- added link left_thumb, mass 0.000009; collision mesh filename=mesh/finger.stl; visual mesh filename=mesh/finger.stl
- link endeffectol: geometry visual cylinder length=0.05 radius=0.002
Joints:
- added joint l_thumb_x: type revolute, parent left_palm, child l_thumb_intermediate_link, origin xyz=-0.008 -0.020 -0.028 rpy=0.3 1 1.4, axis 2 1 0, limit lower=-2.57 upper=0 effort=30 velocity=1
- added joint l_thumb_z: type revolute, parent l_thumb_intermediate_link, child left_thumb, origin xyz=0 0 0 rpy=0 0 0, axis 0 1 0, limit lower=-2.57 upper=0 effort=30 velocity=1
- joint endeffectol_joint: origin xyz=0.00 -0.02 -0.11 rpy=0 0 0 -> xyz=-0.03 0.0 -0.05 rpy=3.14 1.57 -3.14

Commit message: grasper pdate - left hand model fixes - WIP - example for both hands top and side grasp scripts

File: nico_grasper.urdf (robot description, URDF)
Before this commit: robot nico_upper_rh6d, 29 links, 28 joints
Joints:
- joint l_shoulder_z: limit lower=-1.3963 upper=0.4363 effort=30 velocity=1 -> lower=-0.4363 upper=1.3963 effort=30 velocity=1
