Commit message: new methods - lookat and point - urdf ight update

File: urdf/nico_grasper.urdf (robot description, URDF)
Before this commit: robot nico_upper_rh6d, 29 links, 28 joints
Links:
- link sight: geometry visual cylinder length=0.03 radius=0.001

Commit message: bugfix hed_y limits i real robot - urdf modified - WORKAROUND

File: urdf/nico_grasper.urdf (robot description, URDF)
Before this commit: robot nico_upper_rh6d, 29 links, 28 joints
Joints:
- joint head_y: limit lower=-0.8726 upper=0.4363 effort=30 velocity=1 -> lower=-1.483 upper=0 effort=30 velocity=1; origin xyz=0 0.0 0.105 rpy=0 0 0 -> xyz=0 0.0 0.105 rpy=0 -0.69 0

Commit message: urdf and json config updated after repositioning the head to correct position

File: urdf/nico_grasper.urdf (robot description, URDF)
Before this commit: robot nico_upper_rh6d, 29 links, 28 joints
Joints:
- joint head_y: limit lower=-1.483 upper=0 effort=30 velocity=1 -> lower=-0.8726 upper=0.4363 effort=30 velocity=1; origin xyz=0 0.0 0.105 rpy=0 -0.69 0 -> xyz=0 0.0 0.105 rpy=0 0 0
